File: BluePill-Relay-Carrier.kicad_pcb (KiCad board)
At the start: 4 copper layers, 80 x 70 mm, 25 parts, among them J1 5V_IN, J2 RY1_OUT, J3 RY2_OUT, J4 SENSOR, Q1 2N3904, Q2 2N3904, U1 Bluepill_L, U2 Bluepill_R

Commit message: auto-backup 2026-07-18 22:26:17
Parts:
- moved R4 91.5 mm to (76.0, 51.0), turned to -90 degrees
- moved D5 90.4 mm to (76.0, 49.0), turned to 90 degrees
- moved J3 84.2 mm to (57.0, 62.0)
- moved R3 77.7 mm to (76.0, 16.0), turned to -90 degrees
- moved D4 77.3 mm to (76.0, 14.0), turned to 90 degrees
- moved RY2 71.2 mm to (56.0, 44.0)
- moved U2 68.5 mm to (50.0, 46.9), turned to -90 degrees
- moved J4 67.2 mm to (26.0, 62.0)
- moved R2 65.2 mm to (38.0, 53.0)
- moved J2 64.4 mm to (57.0, 30.0)
- moved D2 63.5 mm to (8.00, 63.0)
- moved C2 59.9 mm to (28.0, 53.0)
- moved C1 57.9 mm to (18.0, 55.0), turned to 90 degrees
- moved RY1 56.9 mm to (56.0, 10.0)
- moved U1 55.5 mm to (50.0, 24.0), turned to -90 degrees
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Routing:
- net RY2_Drive: track 0.00 -> 77.0 mm
- net RY1_Drive: track 0.00 -> 71.4 mm, vias 0 -> 1
- net PA1: track 0.00 -> 52.3 mm, vias 0 -> 1
- net Q2B: track 0.00 -> 42.4 mm
- net VCC_IN: track 0.00 -> 23.6 mm
- net RY1_NC: track 0.00 -> 22.0 mm
- net Q1B: track 0.00 -> 22.0 mm
- net RY2_NC: track 0.00 -> 19.0 mm
- net PB7: track 0.00 -> 16.7 mm
- net RY1_COM: track 0.00 -> 15.9 mm
- net PB6: track 0.00 -> 15.7 mm
- net RY2_NO: track 0.00 -> 15.1 mm
- net RY2_COM: track 0.00 -> 13.2 mm
- net PA0: track 0.00 -> 13.2 mm
- net RY1_NO: track 0.00 -> 10.6 mm
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- added copper zone on In2.Cu, net +5V
- added copper zone on In1.Cu, net GND

Commit message: auto-backup 2026-07-19 21:26:19
Parts:
- moved RY2 0.90 mm to (56.0, 43.1)
- moved D5 0.60 mm to (76.0, 48.4)
- moved D4 0.60 mm to (76.0, 13.4)
Changed lines of the file:
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@@
 	(footprint "LED_THT:LED_D3.0mm"
 		(layer "F.Cu")
-		(at 76 49 90)
+		(at 76 48.4 90)
 		(descr "LED, diameter 3.0mm, 2 pins, generated by kicad-footprint-generator")
 		(tags "LED")
@@
 		)
 		(point
-			(at 76 47.73)
+			(at 76 47.13)
 			(size 2)
 			(layer "F.Fab")
@@
 	(footprint "LED_THT:LED_D3.0mm"
 		(layer "F.Cu")
-		(at 76 14 90)
+		(at 76 13.4 90)
 		(descr "LED, diameter 3.0mm, 2 pins, generated by kicad-footprint-generator")
 		(tags "LED")
@@
 		)
 		(point
-			(at 76 12.73)
+			(at 76 12.13)
 			(size 2)
 			(layer "F.Fab")
@@
 	(footprint "Relay_THT:Relay_SPDT_Hongfa_JQC-3FF_0XX-1Z"
 		(layer "F.Cu")
-		(at 56 44)
+		(at 56 43.1)
 		(descr "Hongfa subminature high power latching SPDT relay 5, 6, 9, 12, 18, 24, 48VDC. 10A switching current, Form-B https://www.generationrobots.com/media/JQC-3FF-v1.pdf")
 		(tags "relays Hongmei 1-coil")
